Commit message: add gazebo configuration

File: warehouse_robot/urdf/common_properties.xacro (robot description, xacro)
@@ -1,5 +1,5 @@
 <robot xmlns:xacro="http://www.ros.org/wiki/xacro">
-  <material name="purple">
-    <color rgba="0.42 0.17 0.78 0.8" />
+  <material name="blue">
+    <color rgba="0.157 0.353 0.627 1.0"/>
   </material>
   <material name="grey">

File: warehouse_robot/urdf/mobile_base.xacro (robot description, xacro)
@@ -7,5 +7,5 @@
             </geometry>
             <origin xyz="0 0 0" rpy="0 0 0" />
-            <material name="purple" />
+            <material name="blue" />
         </visual>
         <collision>
@@ -74,4 +74,8 @@
             origin_xyz="0 0 0" origin_rpy="0 0 0" />
     </link>
+    <gazebo reference="caster_wheel_link">
+        <mu1>0.0</mu1>
+        <mu2>0.0</mu2>
+    </gazebo>
     <joint name="footprint_base_joint" type="fixed">
         <parent link="base_footprint" />
@@ -84,5 +88,5 @@
         <origin xyz="-${chassis_length/4} -${wheel_seperation_from_center} -${chassis_height/2}"
             rpy="${pi/2} 0 0" />
-        <axis xyz="0 0 1" />
+        <axis xyz="0 0 -1" />
     </joint>
     <joint name="base_left_wheel_joint" type="continuous">
@@ -91,5 +95,5 @@
         <origin xyz="-${chassis_length/4} ${wheel_seperation_from_center} -${chassis_height/2}"
             rpy="${pi/2} 0 0" />
-        <axis xyz="0 0 1" />
+        <axis xyz="0 0 -1" />
     </joint>
     <joint name="base_castor_wheel_joint" type="fixed">

File: warehouse_robot/urdf/warehouse_robot.urdf.xacro (robot description, xacro)
@@ -3,3 +3,9 @@
   <xacro:include filename="common_properties.xacro" />
   <xacro:include filename="mobile_base.xacro" />
+  <xacro:include filename="warehouse_robot.control.xacro" />
+  <gazebo>
+    <plugin filename="gz_ros2_control-system" name="gz_ros2_control::GazeboSimROS2ControlPlugin">
+      <parameters>$(find warehouse_robot)/config/diff_control_drive.yaml</parameters>
+    </plugin>
+  </gazebo>
 </robot>

Commit message: add lidar urdf and bridge.

File: warehouse_robot/urdf/common_properties.xacro (robot description, xacro)
@@ -1,8 +1,11 @@
 <robot xmlns:xacro="http://www.ros.org/wiki/xacro">
   <material name="blue">
-    <color rgba="0.157 0.353 0.627 1.0"/>
+    <color rgba="0.157 0.353 0.627 1.0" />
   </material>
   <material name="grey">
     <color rgba="0.5 0.5 0.5 1" />
+  </material>
+  <material name="black">
+    <color rgba="0.0 0.0 0.0 1.0" />
   </material>
   <xacro:property name="chassis_length" value="0.6" />
@@ -15,4 +18,6 @@
   <xacro:property name="wheel_seperation_from_center" value="0.22" />
   <xacro:property name="caster_wheel_radius" value="0.04" />
+  <xacro:property name="lidar_radius" value="0.04"/>
+  <xacro:property name="lidar_length" value="0.08"/>
   <xacro:macro name="box_inertia" params="m x y z origin_xyz origin_rpy">
     <inertial>

File: warehouse_robot/urdf/mobile_base.xacro (robot description, xacro)
@@ -74,4 +74,19 @@
             origin_xyz="0 0 0" origin_rpy="0 0 0" />
     </link>
+    <link name="lidar_link">
+        <visual>
+            <geometry>
+                <cylinder radius="${lidar_radius}" length="${lidar_length}" />
+            </geometry>
+            <origin xyz="0 0 0" rpy="0 0 0" />
+            <material name="black" />
+        </visual>
+        <collision>
+            <geometry>
+                <sphere radius="${caster_wheel_radius}" />
+            </geometry>
+            <origin xyz="0 0 0" rpy="0 0 0" />
+        </collision>
+    </link>
     <gazebo reference="caster_wheel_link">
         <mu1>0.0</mu1>
@@ -104,3 +119,8 @@
             rpy="0 0 0" />
     </joint>
+    <joint name="base_lidar_link" type="fixed">
+        <parent link="base_link" />
+        <child link="lidar_link" />
+        <origin xyz="${chassis_length/4} 0 ${chassis_height/2}" rpy="0 0 0"></origin>
+    </joint>
 </robot>

File: warehouse_robot/urdf/warehouse_robot.urdf.xacro (robot description, xacro)
@@ -9,3 +9,29 @@
     </plugin>
   </gazebo>
+  <gazebo reference="lidar_link">
+    <sensor name="lidar_sensor" type="gpu_lidar">
+        <pose>0 0 0 0 0 0</pose>
+        <frame_id>lidar_link</frame_id>
+        <gz_frame_id>lidar_link</gz_frame_id>
+        <topic>scan</topic>
+        <update_rate>10</update_rate>
+        <lidar>
+            <scan>
+                <horizontal>
+                    <samples>360</samples>
+                    <resolution>1</resolution>
+                    <min_angle>-${pi}</min_angle>
+                    <max_angle>${pi}</max_angle>
+                </horizontal>
+            </scan>
+            <range>
+                <min>0.10</min>
+                <max>12.0</max>
+                <resolution>0.01</resolution>
+            </range>
+        </lidar>
+        <always_on>true</always_on>
+        <visualize>true</visualize>
+    </sensor>
+</gazebo>
 </robot>
